File: hardware/ithowifi_4l.sch (KiCad schematic (older format))
At the start: 32 parts, among them J1 CONN_01X07, J2 conn, J3 Conn_Coaxial, J4 TC2030-MCP-NL, Q1 BSS138, Q2 BSS138, U1 ESP32-WROOM, U2 CC1101-868MHz-Module, U3 AMS1117-3.3

Commit message: Update PCB files Change C to HTML Celcius Small CC1101 lib cleanup Update attiny firmware files
Parts:
- added J5: Conn_02x02_Odd_Even, Connector_PinHeader_2.54mm:PinHeader_2x02_P2.54mm_Vertical, symbol Connector_Generic:Conn_02x02_Odd_Even
Connections:
- net +3V3: now also J5.2 (Pin_2)
- net GND: now also J5.4 (Pin_4)
- net SCL_L: now also J5.1 (Pin_1)
- net SDA_L: now also J5.3 (Pin_3)
Changed lines of the file:
@@
 Connection ~ 8875 5225
 Wire Wire Line
-	11475 5225 13625 5225
+	11475 5225 12925 5225
 Wire Wire Line
 	7725 4250 7725 5225
@@
 	5775 3900 5750 3900
 Connection ~ 5775 3900
+Wire Wire Line
+	11975 4150 11975 4975
+Connection ~ 11975 4150
+Wire Wire Line
+	12125 3950 12125 4875
+Wire Wire Line
+	12125 4875 12200 4875
+Connection ~ 12125 3950
+$Comp
+L power:+3V3 #PWR0106
+U 1 1 605DB0AB
+P 12925 4650
+F 0 "#PWR0106" H 12925 4500 50  0001 C CNN
+F 1 "+3V3" H 12940 4823 50  0000 C CNN
+F 2 "" H 12925 4650 50  0001 C CNN
+F 3 "" H 12925 4650 50  0001 C CNN
+	1    12925 4650
+	1    0    0    -1
+$EndComp
+Wire Wire Line
+	12700 4875 12925 4875
+Wire Wire Line
+	12925 4650 12925 4875
+Wire Wire Line
+	12700 4975 12925 4975
+Wire Wire Line
+	12925 4975 12925 5225
+Connection ~ 12925 5225
+Wire Wire Line
+	12925 5225 13625 5225
+$Comp
+L Connector_Generic:Conn_02x02_Odd_Even J5
+U 1 1 605C151F
+P 12400 4875
+F 0 "J5" H 12450 5092 50  0000 C CNN
+F 1 "Conn_02x02_Odd_Even" H 12450 5001 50  0000 C CNN
+F 2 "Connector_PinHeader_2.54mm:PinHeader_2x02_P2.54mm_Vertical" H 12400 4875 50  0001 C CNN
+F 3 "~" H 12400 4875 50  0001 C CNN
+	1    12400 4875
+	1    0    0    -1
+$EndComp
+Wire Wire Line
+	11975 4975 12200 4975
 $EndSCHEMATC
