File: hardware/ithowifi_4l.kicad_pcb (KiCad board)
At the start: 4 copper layers, 42.3 x 51.5 mm, 34 parts, among them J1 CONN_01X07, J2 conn, J3 Conn_Coaxial, J4 TC2030-MCP-NL, J5 Conn_02x02_Odd_Even, Q1 BSS138, Q2 BSS138, U1 ESP32-WROOM, U2 CC1101-868MHz-Module, U3 AMS1117-3.3

Commit message: Hardware files for v2.6 and v2.7
Parts:
- removed H1: MountingHole, MountingHole:MountingHole_2.5mm
- removed JP1: Failsafe, Jumper:SolderJumper-2_P1.3mm_Open_RoundedPad1.0x1.5mm
- removed U3: AMS1117-3.3, Package_TO_SOT_SMD:SOT-223-3_TabPin2
- added SW1: Fail safe, Button_Switch_SMD:SW_SPST_PTS810, F.Cu at (119.8, 110.5)
- C4: value 10uF -> 470uF; footprint Capacitor_Tantalum_SMD:CP_EIA-3216-12_Kemet-S -> Capacitor_SMD:C_Elec_6.3x7.7
- C6: footprint Capacitor_Tantalum_SMD:CP_EIA-3216-12_Kemet-S -> Capacitor_SMD:C_0805_2012Metric
- R10, R7, R8: value 10K -> R10K
- moved C4 15.5 mm to (111.6, 129.2), turned to 90 degrees
- moved J4 11.1 mm to (92.0, 107.9), turned to 90 degrees
- moved R7 11.0 mm to (89.4, 119.7)
- moved C2 10.9 mm to (91.7, 119.7), turned to 90 degrees
- moved R5 9.07 mm to (113.7, 117.6), turned to 270 degrees
- moved LED2 8.14 mm to (111.1, 117.6), turned to 270 degrees
- moved D1 6.41 mm to (94.2, 120.4), turned to 270 degrees
- moved C6 5.46 mm to (113.5, 137.8)
- moved ATtiny1614 5.40 mm to (103.0, 121.0)
- moved C1 5.40 mm to (97.1, 121.1)
- moved R10 0.27 mm to (105.4, 127.2)
- renumbered R-78E5.0 to R-78E3.0
Connections:
- C6 pad 1: +5V -> +15V
- J2 pad 2: +16V3 -> +15V
- J2 pad 6: Net-(J2-Pad6) -> +5V
- R-78E3.0 pad 1: +16V3 -> +15V
- R-78E3.0 pad 3: +5V -> +3V3
Routing:
- net Net-(R10-Pad2): track 13.2 -> 33.7 mm, vias 0 -> 2
- net +5V: track 32.3 -> 13.5 mm, vias 4 -> 2
- net EN: track 29.1 -> 45.1 mm
- net UPDI: track 28.3 -> 43.6 mm, vias 1 -> 2
- net +3V3: track 29.8 -> 43.6 mm, vias 18 -> 15
- net +15V: track 0.00 -> 11.0 mm
- net DTR: track 30.9 -> 22.3 mm, vias 2 -> 1
- net SCL_L: track 77.0 -> 85.6 mm, vias 3 -> 2
- net Net-(ATtiny1614-Pad4): track 35.7 -> 28.4 mm, vias 0 -> 2
- net +16V3: track 5.88 -> 0.00 mm
- net GND: track 10.8 -> 15.5 mm
- net D1/TX0: track 48.5 -> 44.1 mm
- net SDA_L: track 90.5 -> 93.2 mm, vias 4 -> 2
- net D0: track 14.9 -> 17.3 mm
- net Net-(ATtiny1614-Pad11): track 11.7 -> 10.2 mm
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- removed copper zone on F.Cu, net +3V3
Other:
- board text added: "5V"
- board text added: "Itho CVE ESP WiFi Controller v2.7 Arjen Hiemstra - GNU GPL 3.0"
- board text removed: "Itho CVE ESP WiFi Controller v2.5 Arjen Hiemstra - GNU GPL 3.0"

Commit message: Update hardware files
Parts:
- removed REF**: Pin_D1.0mm_L10.0mm, Connector_Pin:Pin_D1.0mm_L10.0mm
- added C3: 10uF, Capacitor_SMD:C_0805_2012Metric, F.Cu at (108.4, 142.4)
- added D2: D_Schottky, Diode_SMD:D_SOD-123, F.Cu at (109.8, 146.1)
- added R11: R1K, Resistor_SMD:R_0805_2012Metric, F.Cu at (111.2, 142.4)
- D1: value D_Zener -> D_Schottky
- moved C5 1.38 mm to (110.4, 148.8)
- moved D1 0.07 mm to (94.3, 120.4)
- renumbered R-78E3.0 to R-78E3.3
Connections:
- net EN renamed Net-(C2-Pad1)
Routing:
- net Net-(C3-Pad1): track 0.00 -> 4.32 mm
- net +3V3: track 43.6 -> 47.8 mm
- net Net-(C2-Pad1): track 45.1 -> 47.6 mm
Other:
- board text added: "Itho CVE ESP WiFi Controller v2.8 Arjen Hiemstra - GNU GPL 3.0"
- board text removed: "Itho CVE ESP WiFi Controller v2.7 Arjen Hiemstra - GNU GPL 3.0"
