File: hardware/non-cve wifi module/ithowifi_4l.kicad_sch (KiCad schematic)
At the start: 46 parts, among them J1 USB_B_Micro, J2 RJ45_LED_Shielded, J4 Conn_02x02_Odd_Even, J5 Conn_02x02_Odd_Even, Q1 BSS138, Q2 BSS138, Q3 BC847, Q4 BC847, SW1 Fail safe, SW2 Reset, U1 ESP32-WROOM, U2 CC1101-868MHz-Module, U3 CH340G, U4 AMS1117-3.3, Y1 Crystal_GND24_Small

Commit message: update hardware files
Parts:
- removed C5: 0.1uF, Capacitor_SMD:C_0805_2012Metric, symbol Device:C
- removed R-78E5.0: U2, Converter_DCDC:Converter_DCDC_RECOM_R-78E-0.5_THT, symbol Regulator_Switching:R-78E5.0-0.5
- added C11: 10uF, Capacitor_SMD:C_0805_2012Metric, symbol Device:C
- added U5: 780xMT, nrg_watch:Mornsun 780xMT, symbol nrgwatch:780xMT
- C3: value 10uF -> 22uF
Connections:
- net +15V: now also U5.1 (Vin), U5.6 (Ctrl)
- net +5V: now also C11.1, U5.3 (Vout)
- net GND: now also C11.2, U5.2 (GND), U5.5 (GND)
- no-connect marks 27 -> 28
Other:
- moved on the sheet: C4, C7, U4

Commit message: Update hardware files
Parts:
- C4: footprint Capacitor_SMD:C_Elec_6.3x7.7 -> Capacitor_Tantalum_SMD:CP_EIA-7343-31_Kemet-D; LCSC C134738 -> C7229
Changed lines of the file:
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@@
       (effects (font (size 1.27 1.27)) (justify left))
     )
-    (property "Footprint" "Capacitor_SMD:C_Elec_6.3x7.7" (id 2) (at 291.1602 156.21 0)
+    (property "Footprint" "Capacitor_Tantalum_SMD:CP_EIA-7343-31_Kemet-D" (id 2) (at 291.1602 156.21 0)
       (effects (font (size 1.27 1.27)) hide)
     )
@@
       (effects (font (size 1.27 1.27)) hide)
     )
-    (property "LCSC" "C134738" (id 4) (at 290.195 152.4 0)
+    (property "LCSC" "C7229" (id 4) (at 290.195 152.4 0)
       (effects (font (size 1.27 1.27)) hide)
     )
@@
     )
     (path "/00000000-0000-0000-0000-00005fbf514b"
-      (reference "C4") (unit 1) (value "470uF") (footprint "Capacitor_SMD:C_Elec_6.3x7.7")
+      (reference "C4") (unit 1) (value "470uF") (footprint "Capacitor_Tantalum_SMD:CP_EIA-7343-31_Kemet-D")
     )
     (path "/00000000-0000-0000-0000-00005fe55ec6"
