File: hardware/non-cve wifi module/ithowifi_4l.kicad_pcb (KiCad board)
At the start: 4 copper layers, 63.1 x 49.8 mm, 46 parts, among them J1 USB_B_Micro, J2 RJ45_LED_Shielded, J4 Conn_02x02_Odd_Even, J5 Conn_02x02_Odd_Even, Q1 BSS138, Q2 BSS138, Q3 BC847, Q4 BC847, SW1 Fail safe, SW2 Reset, U1 ESP32-WROOM, U2 CC1101-868MHz-Module, U3 CH340G, U4 AMS1117-3.3, U5 R-78E5.0, Y1 Crystal_GND24_Small

Commit message: update hardware files
Parts:
- removed C5: 0.1uF, Capacitor_SMD:C_0805_2012Metric
- added C11: 10uF, Capacitor_SMD:C_0805_2012Metric, F.Cu at (83.8, 116.2)
- C3: value 10uF -> 22uF
- U5: value R-78E5.0 -> 780xMT; footprint Converter_DCDC:Converter_DCDC_RECOM_R-78E-0.5_THT -> nrg_watch:Mornsun 780xMT
- moved C3 16.4 mm to (80.6, 132.3)
- moved U5 3.59 mm to (74.2, 134.1)
- moved C6 1.68 mm to (80.6, 136.0), turned to 90 degrees
Routing:
- net GND: track 4.73 -> 14.8 mm, vias 50 -> 57
- net D16_SYS_STATUS: track 32.3 -> 28.5 mm, vias 1 -> 0
- net D17_WIFI_STATUS: track 28.7 -> 31.3 mm
- net +5V: track 77.8 -> 76.6 mm, vias 4 -> 6
- net Net-(J2-Pad12): track 6.84 -> 5.93 mm
- net D0/RX0: track 54.6 -> 54.0 mm, vias 0 -> 2
- net D1/TX0: track 61.1 -> 60.6 mm, vias 0 -> 2
- net +15V: track 29.9 -> 30.1 mm, vias 0 -> 2
Other:
- board text added: "HW rev.: 1 Batch: 10-623"
- board text removed: "HW rev.: 1 Batch: 09-4922"

Commit message: Update hardware files
Parts:
- C4: footprint Capacitor_SMD:C_Elec_6.3x7.7 -> Capacitor_Tantalum_SMD:CP_EIA-7343-31_Kemet-D
- turned C11 to 90 degrees
Routing:
- net GND: track 14.8 -> 12.0 mm
- net +5V: track 76.6 -> 75.8 mm
- net +3V3: track 41.4 -> 40.8 mm

Commit message: update hardware files
Other:
- board text added: "HW rev.: 1 Batch: 12-3823"
- board text removed: "HW rev.: 1 Batch: 10-623"
