File: hardware/cve add-on/ithowifi_4l.kicad_pcb (KiCad board)
At the start: 4 copper layers, 42.3 x 51.5 mm, 33 parts, among them J1 CONN_01X07, J2 conn, J3 Conn_Coaxial, J4 TC2030-MCP-NL, J5 Conn_02x02_Odd_Even, Q1 BSS138, Q2 BSS138, SW1 Fail safe, SW2 Reset, U1 ESP32-WROOM, U2 CC1101-868MHz-Module, U3 780xMT

Commit message: Update hardware files
Parts:
- C4: footprint Capacitor_SMD:C_Elec_6.3x7.7 -> Capacitor_Tantalum_SMD:CP_EIA-7343-31_Kemet-D
Routing:
- net +3V3: track 44.6 -> 45.9 mm, vias 14 -> 13
Other:
- board text added: "HW rev.: 2 Batch: 23-x23"
- board text removed: "HW rev.: 2 Batch: 22-623"

Commit message: Update hardware files
Other:
- board text added: "HW rev.: 2 Batch: 23-1923"
- board text removed: "HW rev.: 2 Batch: 23-x23"

Commit message: update hardware files
Parts:
- removed U2: CC1101-868MHz-Module, nrg_watch:CC1101-868MHz-Module
- added J6: conn, Connector_PinSocket_2.54mm:PinSocket_2x04_P2.54mm_Vertical_SMD, F.Cu at (120.6, 134.0)
- added U4: ~, nrg_watch:E70-433MT14S, B.Cu at (96.3, 122.9)
- C2, C3, C4, C5, C6, D2, Q1, Q2, R1, R10, R11, R2, R3, R4, R5, R7, R8, R9, U1, U3: moved to B.Cu
- J2: footprint Connector_PinSocket_2.54mm:PinSocket_2x04_P2.54mm_Vertical -> Connector_PinSocket_2.54mm:PinSocket_2x04_P2.54mm_Vertical_SMD
- J3: footprint Connector_Coaxial:SMA_Amphenol_132289_EdgeMount -> Connector_Coaxial:U.FL_Molex_MCRF_73412-0110_Vertical
- LED1, LED2: footprint LED_SMD:LED_0805_2012Metric -> nrg_watch:MHT151 counterpost led; moved to B.Cu
- SW1, SW2: footprint nrg_watch:TS-1187 -> nrg_watch:switch YTS1T0022ABJ01; moved to B.Cu
- moved J1 48.6 mm to (114.1, 147.2), turned to 180 degrees
- moved J4 39.3 mm to (108.6, 143.5), turned to 180 degrees
- moved SW1 27.7 mm to (83.0, 115.2)
- moved R11 27.2 mm to (84.6, 136.4), turned to -90 degrees
- moved C5 25.9 mm to (84.6, 149.2), turned to -90 degrees
- moved D2 25.2 mm to (84.6, 144.7), turned to 90 degrees
- moved C3 23.9 mm to (84.6, 140.1), turned to -90 degrees
- moved SW2 21.3 mm to (83.1, 122.2), turned to -90 degrees
- moved R9 20.8 mm to (111.2, 131.6), turned to 90 degrees
- moved LED1 20.5 mm to (109.1, 128.7), turned to 0 degrees
- moved R10 19.4 mm to (87.2, 127.3)
- moved R5 19.1 mm to (84.6, 129.1)
- moved R8 16.6 mm to (109.2, 131.6), turned to -90 degrees
- moved R7 15.8 mm to (84.6, 132.9)
- moved J5 14.7 mm to (110.4, 137.3), turned to 180 degrees
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Routing:
- net SDA_L: track 83.0 -> 2.23 mm, vias 2 -> 0
- net SCL_L: track 70.3 -> 2.24 mm, vias 2 -> 0
- net Net-(D2-A): track 50.2 -> 0.00 mm, vias 2 -> 0
- net +3V3: track 45.9 -> 0.00 mm, vias 13 -> 0
- net D1/TX0: track 43.8 -> 0.00 mm, vias 1 -> 0
- net D0: track 42.2 -> 0.00 mm, vias 1 -> 0
- net D0/RX0: track 41.6 -> 0.00 mm, vias 1 -> 0
- net D23_MOSI: track 33.5 -> 0.00 mm, vias 1 -> 0
- net D18_SCK: track 24.2 -> 0.00 mm, vias 1 -> 0
- net GND: track 22.8 -> 0.00 mm, vias 40 -> 12
- net D19_MISO: track 22.0 -> 0.00 mm, vias 1 -> 0
- net Net-(U1-IO14): track 20.5 -> 0.00 mm
- net D4_IRQ: track 19.0 -> 0.00 mm, vias 1 -> 0
- net D5_SS: track 14.5 -> 0.00 mm, vias 1 -> 0
- net +15V: track 14.5 -> 0.00 mm, vias 0 -> 1
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- added copper zone on In1.Cu, net GND
- removed copper zone on In1.Cu, net +3V3
Other:
- board size 42.3 x 51.5 mm -> 48.2 x 64.5 mm
- board text added: "HW rev.: 2 Batch: 23-2323"
- board text removed: "HW rev.: 2 Batch: 23-1923"
