File: hardware/cve add-on/ithowifi_4l.kicad_sch (KiCad schematic)
At the start: 33 parts, among them J1 CONN_01X07, J2 conn, J3 Conn_Coaxial, J4 TC2030-MCP-NL, J5 Conn_02x02_Odd_Even, Q1 BSS138, Q2 BSS138, SW1 Fail safe, SW2 Reset, U1 ESP32-WROOM, U2 CC1101-868MHz-Module

Commit message: update hardware files
Parts:
- Q1, Q2: footprint Package_TO_SOT_SMD:SOT-23 -> Package_TO_SOT_SMD:SOT-23W
Changed lines of the file:
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@@
     (property "Reference" "Q1" (id 0) (at 258.445 109.1946 90))
     (property "Value" "BSS138" (id 1) (at 258.445 111.506 90))
-    (property "Footprint" "Package_TO_SOT_SMD:SOT-23" (id 2) (at 256.54 107.95 0)
+    (property "Footprint" "Package_TO_SOT_SMD:SOT-23W" (id 2) (at 256.54 107.95 0)
       (effects (font (size 1.27 1.27) italic) (justify left) hide)
     )
@@
     (property "Reference" "Q2" (id 0) (at 272.415 104.1146 90))
     (property "Value" "BSS138" (id 1) (at 272.415 106.426 90))
-    (property "Footprint" "Package_TO_SOT_SMD:SOT-23" (id 2) (at 270.51 102.87 0)
+    (property "Footprint" "Package_TO_SOT_SMD:SOT-23W" (id 2) (at 270.51 102.87 0)
       (effects (font (size 1.27 1.27) italic) (justify left) hide)
     )
@@
     )
     (path "/00000000-0000-0000-0000-00005e6ce08c"
-      (reference "Q1") (unit 1) (value "BSS138") (footprint "Package_TO_SOT_SMD:SOT-23")
+      (reference "Q1") (unit 1) (value "BSS138") (footprint "Package_TO_SOT_SMD:SOT-23W")
     )
     (path "/00000000-0000-0000-0000-00005e6d9a33"
-      (reference "Q2") (unit 1) (value "BSS138") (footprint "Package_TO_SOT_SMD:SOT-23")
+      (reference "Q2") (unit 1) (value "BSS138") (footprint "Package_TO_SOT_SMD:SOT-23W")
     )
     (path "/00000000-0000-0000-0000-00005e596dc0"

Commit message: update hardware files
Parts:
- removed R-78E3.3: U2, Converter_DCDC:Converter_DCDC_RECOM_R-78E-0.5_THT, symbol Regulator_Switching:R-78E5.0-0.5
- added U3: 780xMT, nrg_watch:Mornsun 780xMT, symbol nrgwatch:780xMT
Connections:
- net +15V: now also U3.1 (Vin), U3.6 (Ctrl)
- net +3V3: now also U3.3 (Vout)
- net GND: now also U3.2 (GND), U3.5 (GND)
- no-connect marks 1 -> 2

Commit message: Update hardware files
Parts:
- C4: footprint Capacitor_SMD:C_Elec_6.3x7.7 -> Capacitor_Tantalum_SMD:CP_EIA-7343-31_Kemet-D; LCSC C134738 -> C7229
Changed lines of the file:
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@@
       (effects (font (size 1.27 1.27)) (justify left))
     )
-    (property "Footprint" "Capacitor_SMD:C_Elec_6.3x7.7" (id 2) (at 87.3252 183.515 0)
+    (property "Footprint" "Capacitor_Tantalum_SMD:CP_EIA-7343-31_Kemet-D" (id 2) (at 87.3252 183.515 0)
       (effects (font (size 1.27 1.27)) hide)
     )
@@
       (effects (font (size 1.27 1.27)) hide)
     )
-    (property "LCSC" "C134738" (id 4) (at 86.36 179.705 0)
+    (property "LCSC" "C7229" (id 4) (at 86.36 179.705 0)
       (effects (font (size 1.27 1.27)) hide)
     )
@@
     )
     (path "/00000000-0000-0000-0000-00005fbf514b"
-      (reference "C4") (unit 1) (value "470uF") (footprint "Capacitor_SMD:C_Elec_6.3x7.7")
+      (reference "C4") (unit 1) (value "470uF") (footprint "Capacitor_Tantalum_SMD:CP_EIA-7343-31_Kemet-D")
     )
     (path "/00000000-0000-0000-0000-00005fbf513f"

Commit message: update hardware files
Parts:
- removed U2: CC1101-868MHz-Module, nrg_watch:CC1101-868MHz-Module, symbol nrg_watch:CC1101-868MHz-Module
- added J6: conn, Connector_PinSocket_2.54mm:PinSocket_2x04_P2.54mm_Vertical_SMD, symbol Connector_Generic:Conn_02x04_Odd_Even
- added U4: ~, nrg_watch:E70-433MT14S, symbol nrg_watch:EByte_E07_CC1101
- J2: footprint Connector_PinSocket_2.54mm:PinSocket_2x04_P2.54mm_Vertical -> Connector_PinSocket_2.54mm:PinSocket_2x04_P2.54mm_Vertical_SMD
- J3: footprint Connector_Coaxial:SMA_Amphenol_132289_EdgeMount -> Connector_Coaxial:U.FL_Molex_MCRF_73412-0110_Vertical
- LED1, LED2: footprint LED_SMD:LED_0805_2012Metric -> nrg_watch:MHT151 counterpost led
- SW1, SW2: footprint nrg_watch:TS-1187 -> nrg_watch:switch YTS1T0022ABJ01
Connections:
- net +15V: now also J6.1 (Pin_1)
- net +3V3: now also U4.1 (VCC)
- net +5V: now also J6.5 (Pin_5)
- net D18_SCK: now also U4.15 (SCK)
- net D19_MISO: now also U4.12 (MISO/GDO1)
- net D23_MOSI: now also U4.13 (MOSI)
- net D4_IRQ: now also U4.20 (GDO2)
- net D5_SS: now also U4.14 (CSN)
- net GND: now also J6.6 (Pin_6), U4.16 (GND), U4.2 (GND), U4.7 (GND)
- net SCL: now also J6.7 (Pin_7)
- net SDA: now also J6.8 (Pin_8)
- net at H1.1, J3.1 (In): now also U4.6 (ANT)
- no-connect marks 2 -> 4
Other:
- moved on the sheet: H1, J3
