File: hardware/cve add-on/ithowifi_4l_v21_tht.kicad_pcb (KiCad board)
At the start: 4 copper layers, 42.3 x 51.5 mm, 33 parts, among them J1 CONN_01X07, J2 conn, J3 Conn_Coaxial, J4 TC2030-MCP-NL, J5 Conn_02x02_Odd_Even, Q1 BSS138, Q2 BSS138, SW1 Fail safe, SW2 Reset, U1 ESP32-WROOM, U2 CC1101-868MHz-Module, U3 780xMT

Commit message: update hardware files
Parts:
- removed U3: 780xMT, nrg_watch:Mornsun 780xMT
- added R-78E3.3: U2, Converter_DCDC:Converter_DCDC_RECOM_R-78E-0.5_THT, F.Cu at (121.3, 143.0)
- moved C6 1.23 mm to (113.5, 137.8)
Routing:
- net GND: track 23.3 -> 15.4 mm, vias 40 -> 38
- net +15V: track 14.5 -> 11.0 mm
- net +3V3: track 44.6 -> 41.8 mm, vias 14 -> 13
Other:
- board text added: "HW rev.: 2 Batch: 21-623"
- board text removed: "HW rev.: 2 Batch: 22-623"

Commit message: Update hardware files
Parts:
- removed R-78E3.3: U2, Converter_DCDC:Converter_DCDC_RECOM_R-78E-0.5_THT
- added U3: R-78E3.3-0.5, Converter_DCDC:Converter_DCDC_RECOM_R-78E-0.5_THT, F.Cu at (121.3, 143.0)
- C4: footprint Capacitor_SMD:C_Elec_6.3x7.7 -> Capacitor_Tantalum_SMD:CP_EIA-7343-31_Kemet-D
Routing:
- net +3V3: track 41.8 -> 43.1 mm, vias 13 -> 12
- net GND: track 15.4 -> 14.8 mm
Other:
- board text added: "HW rev.: 2 Batch: 24-1923"
- board text removed: "HW rev.: 2 Batch: 21-623"

Commit message: update hardware files
Other:
- board text added: "HW rev.: 2 Batch: 21-2323"
- board text removed: "HW rev.: 2 Batch: 24-1923"
