File: hardware/cve add-on/ithowifi_4l_v21_tht.kicad_sch (KiCad schematic)
At the start: 33 parts, among them J1 CONN_01X07, J2 conn, J3 Conn_Coaxial, J4 TC2030-MCP-NL, J5 Conn_02x02_Odd_Even, Q1 BSS138, Q2 BSS138, SW1 Fail safe, SW2 Reset, U1 ESP32-WROOM, U2 CC1101-868MHz-Module, U3 R-78E3.3-0.5

Commit message: update hardware files
Connections:
- no-connect marks 2 -> 15
Changed lines of the file:
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@@
   (junction (at 146.685 91.44) (diameter 0) (color 0 0 0 0)
   )
-  (no_connect (at 70.485 128.27))
+  (no_connect (at 174.625 118.11))
+  (no_connect (at 193.675 97.79))
+  (no_connect (at 182.245 118.11))
   (no_connect (at 53.975 88.9))
+  (no_connect (at 169.545 118.11))
+  (no_connect (at 146.685 83.82))
+  (no_connect (at 146.685 81.28))
+  (no_connect (at 146.685 106.68))
+  (no_connect (at 177.165 118.11))
+  (no_connect (at 172.085 118.11))
+  (no_connect (at 167.005 118.11))
+  (no_connect (at 146.685 86.36))
+  (no_connect (at 164.465 118.11))
+  (no_connect (at 146.685 88.9))
+  (no_connect (at 146.685 101.6))
   (wire (pts (xy 313.69 113.665) (xy 313.69 116.205))
     (stroke (width 0) (type default))
@@
     (stroke (width 0) (type default))
   )
+  (wire (pts (xy 68.58 179.07) (xy 68.58 188.595))
+    (stroke (width 0) (type default))
+  )
   (wire (pts (xy 86.36 188.595) (xy 100.965 188.595))
     (stroke (width 0) (type default))
@@
     (stroke (width 0) (type default))
   )
-  (wire (pts (xy 68.58 179.07) (xy 68.58 188.595))
-    (stroke (width 0) (type default))
-  )
   (wire (pts (xy 245.745 198.755) (xy 245.745 195.58))
     (stroke (width 0) (type default))
@@
     (stroke (width 0) (type default))
   )
+  (wire (pts (xy 50.165 188.595) (xy 68.58 188.595))
+    (stroke (width 0) (type default))
+  )
   (wire (pts (xy 225.425 137.795) (xy 225.425 132.715))
     (stroke (width 0) (type default))
@@
     (stroke (width 0) (type default))
   )
-  (wire (pts (xy 50.165 188.595) (xy 68.58 188.595))
-    (stroke (width 0) (type default))
-  )
